Commit message: update

File: universal_robot/ur_description/urdf/ur5.urdf.xacro (robot description, xacro)
@@ -74,5 +74,11 @@
      wrist_2_lower_limit:=${-pi}    wrist_2_upper_limit:=${pi}
      wrist_3_lower_limit:=${-pi}    wrist_3_upper_limit:=${pi}">
-    <link name="${prefix}base_link" >
+ <!--       new add       -->
+  <joint name="mid_mount_ur_joint" type="fixed">
+    <origin xyz="0.28 0.0 0" rpy="0.0 0.0 -1.5708" />
+    <parent link="mid_mount"/>
+    <child link="mid_mount_ur" />
+  </joint>
+    <link name="${prefix}mid_mount_ur" >
       <visual>
         <geometry>
@@ -93,5 +99,5 @@
     </link>
     <joint name="${prefix}shoulder_pan_joint" type="revolute">
-      <parent link="${prefix}base_link" />
+      <parent link="${prefix}mid_mount_ur" />
       <child link = "${prefix}shoulder_link" />
       <origin xyz="0.0 0.0 ${shoulder_height}" rpy="0.0 0.0 0.0" />
@@ -301,5 +307,5 @@
       -->
       <origin xyz="0 0 0" rpy="0 0 ${-pi}"/>
-      <parent link="${prefix}base_link"/>
+      <parent link="${prefix}mid_mount_ur"/>
       <child link="${prefix}base"/>
     </joint>

File: universal_robot/ur_description/urdf/ur5_joint_limited_robot.urdf.xacro (robot description, xacro)
@@ -15,9 +15,11 @@
     wrist_3_lower_limit="${-pi}" wrist_3_upper_limit="${pi}"
   />
-  <link name="world" />
-  <joint name="world_joint" type="fixed">
-    <parent link="world" />
-    <child link = "base_link" />
+<!--
+  <link name="mid_mount_1" />
+  <joint name="mid_mount_joint_1" type="fixed">
+    <parent link="mid_mount" />
+    <child link = "mid_mount_1" />
     <origin xyz="0.0 0.0 0.0" rpy="0.0 0.0 0.0" />
   </joint>
+-->
 </robot>

Commit message: update

File: universal_robot/ur_description/urdf/ur5.urdf.xacro (robot description, xacro)
@@ -80,5 +80,5 @@
     <child link="mid_mount_ur" />
   </joint>
-    <link name="${prefix}mid_mount_ur" >
+    <link name="mid_mount_ur" >
       <visual>
         <geometry>
@@ -99,5 +99,5 @@
     </link>
     <joint name="${prefix}shoulder_pan_joint" type="revolute">
-      <parent link="${prefix}mid_mount_ur" />
+      <parent link="mid_mount_ur" />
       <child link = "${prefix}shoulder_link" />
       <origin xyz="0.0 0.0 ${shoulder_height}" rpy="0.0 0.0 0.0" />
@@ -307,5 +307,5 @@
       -->
       <origin xyz="0 0 0" rpy="0 0 ${-pi}"/>
-      <parent link="${prefix}mid_mount_ur"/>
+      <parent link="mid_mount_ur"/>
       <child link="${prefix}base"/>
     </joint>

Commit message: update

File: universal_robot/ur_description/urdf/ur5.urdf.xacro (robot description, xacro)
@@ -75,10 +75,10 @@
      wrist_3_lower_limit:=${-pi}    wrist_3_upper_limit:=${pi}">
  <!--       new add       -->
-  <joint name="mid_mount_ur_joint" type="fixed">
+  <joint name="ur_base_link_joint" type="fixed">
     <origin xyz="0.28 0.0 0" rpy="0.0 0.0 -1.5708" />
     <parent link="mid_mount"/>
-    <child link="mid_mount_ur" />
+    <child link="ur_base_link" />
   </joint>
-    <link name="mid_mount_ur" >
+    <link name="ur_base_link" >
       <visual>
         <geometry>
@@ -99,5 +99,5 @@
     </link>
     <joint name="${prefix}shoulder_pan_joint" type="revolute">
-      <parent link="mid_mount_ur" />
+      <parent link="ur_base_link" />
       <child link = "${prefix}shoulder_link" />
       <origin xyz="0.0 0.0 ${shoulder_height}" rpy="0.0 0.0 0.0" />
@@ -307,5 +307,5 @@
       -->
       <origin xyz="0 0 0" rpy="0 0 ${-pi}"/>
-      <parent link="mid_mount_ur"/>
+      <parent link="ur_base_link"/>
       <child link="${prefix}base"/>
     </joint>

Commit message: update

File: universal_robot/ur_description/urdf/ur5.urdf.xacro (robot description, xacro)
@@ -75,6 +75,7 @@
      wrist_3_lower_limit:=${-pi}    wrist_3_upper_limit:=${pi}">
  <!--       new add       -->
+<!--   <origin xyz="0.28 0.0 0" rpy="0.0 0.0 -1.5708" />    -->
   <joint name="ur_base_link_joint" type="fixed">
-    <origin xyz="0.28 0.0 0" rpy="0.0 0.0 -1.5708" />
+    <origin xyz="0.28 0.0 0" rpy="0.0 0.0 ${-pi/4}" />
     <parent link="mid_mount"/>
     <child link="ur_base_link" />

File: universal_robot/ur_description/urdf/ur5_robotiq.urdf.xacro (robot description, xacro)
@@ -26,5 +26,5 @@
   </link>
   <joint name="robotiq_coupler_joint" type="fixed">
-    <origin xyz="0 0 0.06" rpy="${-pi/2.0} 0 ${-pi}" />
+    <origin xyz="0 0 0.06" rpy="${-pi/2.0} 0 ${-(5*pi)/4}" />
     <parent link="tool0"/>
     <child link="robotiq_coupler"/>
@@ -44,5 +44,5 @@
   <!-- Attach the robotiq 85 gripper -->
   <xacro:robotiq_hand prefix="" parent="robotiq_coupler" >
-    <origin xyz="0 0 0.004" rpy="0 ${-pi/2} ${pi}"/>
+    <origin xyz="0 0 0.004" rpy="0 ${0} ${pi}"/>
   </xacro:robotiq_hand>
   <!-- Gazebo FT sensor plugin -->

Commit message: update

File: universal_robot/ur_description/urdf/ur5.urdf.xacro (robot description, xacro)
@@ -136,5 +136,5 @@
       <axis xyz="0 1 0" />
       <xacro:unless value="${joint_limited}">
-        <limit lower="${-2.0 * pi}" upper="${2.0 * pi}" effort="150.0" velocity="3.15"/>
+        <limit lower="${pi/4}" upper="${3*pi / 4}" effort="150.0" velocity="3.15"/>
       </xacro:unless>
       <xacro:if value="${joint_limited}">
@@ -167,5 +167,5 @@
       <axis xyz="0 1 0" />
       <xacro:unless value="${joint_limited}">
-        <limit lower="${-pi}" upper="${pi}" effort="150.0" velocity="3.15"/>
+        <limit lower="${-3*pi / 4}" upper="${3*pi / 4}" effort="150.0" velocity="3.15"/>
       </xacro:unless>
       <xacro:if value="${joint_limited}">
@@ -198,5 +198,5 @@
       <axis xyz="0 1 0" />
       <xacro:unless value="${joint_limited}">
-        <limit lower="${-2.0 * pi}" upper="${2.0 * pi}" effort="28.0" velocity="3.2"/>
+        <limit lower="${-5.0 * pi / 4}" upper="${pi / 4}" effort="28.0" velocity="3.2"/>
       </xacro:unless>
       <xacro:if value="${joint_limited}">
@@ -229,5 +229,5 @@
       <axis xyz="0 0 1" />
       <xacro:unless value="${joint_limited}">
-        <limit lower="${-2.0 * pi}" upper="${2.0 * pi}" effort="28.0" velocity="3.2"/>
+        <limit lower="${10 * pi / 9.0}" upper="${2.0 * pi}" effort="28.0" velocity="3.2"/>
       </xacro:unless>
       <xacro:if value="${joint_limited}">

Commit message: update ur5.urdf.xacro

File: universal_robot/ur_description/urdf/ur5.urdf.xacro (robot description, xacro)
@@ -3,59 +3,59 @@
   <xacro:include filename="$(find ur_description)/urdf/ur.transmission.xacro" />
   <xacro:include filename="$(find ur_description)/urdf/ur.gazebo.xacro" />
-  <!-- Inertia parameters -->
-  <xacro:property name="base_mass" value="4.0" />  <!-- This mass might be incorrect -->
-  <xacro:property name="shoulder_mass" value="3.7000" />
-  <xacro:property name="upper_arm_mass" value="8.3930" />
-  <xacro:property name="forearm_mass" value="2.2750" />
-  <xacro:property name="wrist_1_mass" value="1.2190" />
-  <xacro:property name="wrist_2_mass" value="1.2190" />
-  <xacro:property name="wrist_3_mass" value="0.1879" />
-  <xacro:property name="shoulder_cog" value="0.0 0.00193 -0.02561" />
-  <xacro:property name="upper_arm_cog" value="0.0 -0.024201 0.2125" />
-  <xacro:property name="forearm_cog" value="0.0 0.0265 0.11993" />
-  <xacro:property name="wrist_1_cog" value="0.0 0.110949 0.01634" />
-  <xacro:property name="wrist_2_cog" value="0.0 0.0018 0.11099" />
-  <xacro:property name="wrist_3_cog" value="0.0 0.001159 0.0" />
-  <!-- Kinematic model -->
-  <!-- Properties from urcontrol.conf -->
-  <!--
-    DH for UR5:
-    a = [0.00000, -0.42500, -0.39225,  0.00000,  0.00000,  0.0000]
-    d = [0.089159,  0.00000,  0.00000,  0.10915,  0.09465,  0.0823]
-    alpha = [ 1.570796327, 0, 0, 1.570796327, -1.570796327, 0 ]
-    q_home_offset = [0, -1.570796327, 0, -1.570796327, 0, 0]
-    joint_direction = [-1, -1, 1, 1, 1, 1]
-    mass = [3.7000, 8.3930, 2.2750, 1.2190, 1.2190, 0.1879]
-    center_of_mass = [ [0, -0.02561, 0.00193], [0.2125, 0, 0.11336], [0.11993, 0.0, 0.0265], [0, -0.0018, 0.01634], [0, 0.0018,0.01634], [0, 0, -0.001159] ]
-  -->
-  <xacro:property name="ur5_d1" value="0.089159" />
-  <xacro:property name="ur5_a2" value="-0.42500" />
-  <xacro:property name="ur5_a3" value="-0.39225" />
-  <xacro:property name="ur5_d4" value="0.10915" />
-  <xacro:property name="ur5_d5" value="0.09465" />
-  <xacro:property name="ur5_d6" value="0.0823" />
-  <!-- Arbitrary offsets for shoulder/elbow joints -->
-  <xacro:property name="shoulder_offset" value="0.13585" />  <!-- measured from model -->
-  <xacro:property name="elbow_offset" value="-0.1197" /> <!-- measured from model -->
-  <!-- link lengths used in model -->
-  <xacro:property name="shoulder_height" value="${ur5_d1}" />
-  <xacro:property name="upper_arm_length" value="${-ur5_a2}" />
-  <xacro:property name="forearm_length" value="${-ur5_a3}" />
-  <xacro:property name="wrist_1_length" value="${ur5_d4 - elbow_offset - shoulder_offset}" />
-  <xacro:property name="wrist_2_length" value="${ur5_d5}" />
-  <xacro:property name="wrist_3_length" value="${ur5_d6}" />
-  <!--property name="shoulder_height" value="0.089159" /-->
-  <!--property name="shoulder_offset" value="0.13585" /-->  <!-- shoulder_offset - elbow_offset + wrist_1_length = 0.10915 -->
-  <!--property name="upper_arm_length" value="0.42500" /-->
-  <!--property name="elbow_offset" value="0.1197" /-->       <!-- CAD measured -->
-  <!--property name="forearm_length" value="0.39225" /-->
-  <!--property name="wrist_1_length" value="0.093" /-->     <!-- CAD measured -->
-  <!--property name="wrist_2_length" value="0.09465" /-->   <!-- In CAD this distance is 0.930, but in the spec it is 0.09465 -->
-  <!--property name="wrist_3_length" value="0.0823" /-->
-  <xacro:property name="shoulder_radius" value="0.060" />   <!-- manually measured -->
-  <xacro:property name="upper_arm_radius" value="0.054" />  <!-- manually measured -->
-  <xacro:property name="elbow_radius" value="0.060" />      <!-- manually measured -->
-  <xacro:property name="forearm_radius" value="0.040" />    <!-- manually measured -->
-  <xacro:property name="wrist_radius" value="0.045" />      <!-- manually measured -->
+    <!-- Inertia parameters -->
+    <xacro:property name="base_mass" value="4.0" />  <!-- This mass might be incorrect -->
+    <xacro:property name="shoulder_mass" value="3.7000" />
+    <xacro:property name="upper_arm_mass" value="8.3930" />
+    <xacro:property name="forearm_mass" value="2.2750" />
+    <xacro:property name="wrist_1_mass" value="1.2190" />
+    <xacro:property name="wrist_2_mass" value="1.2190" />
+    <xacro:property name="wrist_3_mass" value="0.1879" />
+     <xacro:property name="shoulder_cog" value="0.0 0.00193 -0.02561" />
+    <xacro:property name="upper_arm_cog" value="0.0 -0.024201 0.2125" />
+    <xacro:property name="forearm_cog" value="0.0 0.0265 0.11993" />
+    <xacro:property name="wrist_1_cog" value="0.0 0.110949 0.01634" />
+    <xacro:property name="wrist_2_cog" value="0.0 0.0018 0.11099" />
+    <xacro:property name="wrist_3_cog" value="0.0 0.001159 0.0" />
+     <!-- Kinematic model -->
+    <!-- Properties from urcontrol.conf -->
+    <!--
+      DH for UR5:
+      a = [0.00000, -0.42500, -0.39225,  0.00000,  0.00000,  0.0000]
+      d = [0.089159,  0.00000,  0.00000,  0.10915,  0.09465,  0.0823]
+      alpha = [ 1.570796327, 0, 0, 1.570796327, -1.570796327, 0 ]
+      q_home_offset = [0, -1.570796327, 0, -1.570796327, 0, 0]
+      joint_direction = [-1, -1, 1, 1, 1, 1]
+      mass = [3.7000, 8.3930, 2.2750, 1.2190, 1.2190, 0.1879]
+      center_of_mass = [ [0, -0.02561, 0.00193], [0.2125, 0, 0.11336], [0.11993, 0.0, 0.0265], [0, -0.0018, 0.01634], [0, 0.0018,0.01634], [0, 0, -0.001159] ]
+    -->
+    <xacro:property name="d1" value="0.089159" />
+    <xacro:property name="a2" value="-0.42500" />
+    <xacro:property name="a3" value="-0.39225" />
+    <xacro:property name="d4" value="0.10915" />
+    <xacro:property name="d5" value="0.09465" />
+    <xacro:property name="d6" value="0.0823" />
+     <!-- Arbitrary offsets for shoulder/elbow joints -->
+    <xacro:property name="shoulder_offset" value="0.13585" />  <!-- measured from model -->
+    <xacro:property name="elbow_offset" value="-0.1197" /> <!-- measured from model -->
+     <!-- link lengths used in model -->
+    <xacro:property name="shoulder_height" value="${d1}" />
+    <xacro:property name="upper_arm_length" value="${-a2}" />
+    <xacro:property name="forearm_length" value="${-a3}" />
+    <xacro:property name="wrist_1_length" value="${d4 - elbow_offset - shoulder_offset}" />
+    <xacro:property name="wrist_2_length" value="${d5}" />
+    <xacro:property name="wrist_3_length" value="${d6}" />
+    <!--property name="shoulder_height" value="0.089159" /-->
+    <!--property name="shoulder_offset" value="0.13585" /-->  <!-- shoulder_offset - elbow_offset + wrist_1_length = 0.10915 -->
+    <!--property name="upper_arm_length" value="0.42500" /-->
+    <!--property name="elbow_offset" value="0.1197" /-->       <!-- CAD measured -->
+    <!--property name="forearm_length" value="0.39225" /-->
+    <!--property name="wrist_1_length" value="0.093" /-->     <!-- CAD measured -->
+    <!--property name="wrist_2_length" value="0.09465" /-->   <!-- In CAD this distance is 0.930, but in the spec it is 0.09465 -->
+    <!--property name="wrist_3_length" value="0.0823" /-->
+     <xacro:property name="shoulder_radius" value="0.060" />   <!-- manually measured -->
+    <xacro:property name="upper_arm_radius" value="0.054" />  <!-- manually measured -->
+    <xacro:property name="elbow_radius" value="0.060" />      <!-- manually measured -->
+    <xacro:property name="forearm_radius" value="0.040" />    <!-- manually measured -->
+    <xacro:property name="wrist_radius" value="0.045" />      <!-- manually measured -->
   <xacro:macro name="cylinder_inertial" params="radius length mass *origin">
     <inertial>
