Commit message: update ur_modern_driver

File: ur_description/urdf/ur5_robotiq.urdf.xacro (robot description, xacro)
@@ -2,5 +2,5 @@
 <robot name="ur5" xmlns:xacro="http://www.ros.org/wiki/xacro">
   <xacro:include filename="$(find ur_description)/urdf/ur5_joint_limited_robot.urdf.xacro" />
-  <xacro:include filename="$(find robotiq_s_model_visualization)/cfg/robotiq_hand_macro.urdf.xacro" />
+  <xacro:include filename="$(find robotiq_3f_gripper_visualization)/cfg/robotiq_hand_macro.urdf.xacro" />
   <!-- Robotiq Coupler -->
   <!--  + Height added by the coupler: 8mm -->
@@ -9,5 +9,5 @@
     <visual>
       <geometry>
-        <mesh filename="package://robotiq_description/meshes/robotiq_85_coupler.stl" />
+        <mesh filename="package://robotiq_3f_gripper_visualization/meshes/robotiq_85_coupler.stl" />
       </geometry>
       <material name="flat_black"/>
@@ -15,5 +15,5 @@
     <collision>
       <geometry>
-        <mesh filename="package://robotiq_description/meshes/robotiq_85_coupler.stl" />
+        <mesh filename="package://robotiq_3f_gripper_visualization/meshes/robotiq_85_coupler.stl" />
       </geometry>
     </collision>
