Commit message: 保存官方版本

File: ur_description/urdf/ur.gazebo.xacro (robot description, xacro)
@@ -1,4 +1,4 @@
 <?xml version="1.0"?>
-<robot xmlns:xacro="http://www.ros.org/wiki/xacro">
+<robot xmlns:xacro="http://wiki.ros.org/xacro">
   <xacro:macro name="ur_arm_gazebo" params="prefix">
     <gazebo reference="${prefix}shoulder_link">

File: ur_description/urdf/ur.transmission.xacro (robot description, xacro)
@@ -1,4 +1,4 @@
 <?xml version="1.0"?>
-<robot xmlns:xacro="http://www.ros.org/wiki/xacro">
+<robot xmlns:xacro="http://wiki.ros.org/xacro">
   <xacro:macro name="ur_arm_transmission" params="prefix">
     <transmission name="${prefix}shoulder_pan_trans">

File: ur_description/urdf/ur5.urdf.xacro (robot description, xacro)
@@ -1,6 +1,22 @@
 <?xml version="1.0"?>
-<robot xmlns:xacro="http://www.ros.org/wiki/xacro">
+<robot xmlns:xacro="http://wiki.ros.org/xacro">
   <xacro:include filename="$(find ur_description)/urdf/ur.transmission.xacro" />
   <xacro:include filename="$(find ur_description)/urdf/ur.gazebo.xacro" />
+  <xacro:macro name="cylinder_inertial" params="radius length mass *origin">
+    <inertial>
+      <mass value="${mass}" />
+      <xacro:insert_block name="origin" />
+      <inertia ixx="${0.0833333 * mass * (3 * radius * radius + length * length)}" ixy="0.0" ixz="0.0"
+        iyy="${0.0833333 * mass * (3 * radius * radius + length * length)}" iyz="0.0"
+        izz="${0.5 * mass * radius * radius}" />
+    </inertial>
+  </xacro:macro>
+  <xacro:macro name="ur5_robot" params="prefix joint_limited
+     shoulder_pan_lower_limit:=${-pi}    shoulder_pan_upper_limit:=${pi}
+     shoulder_lift_lower_limit:=${-pi}    shoulder_lift_upper_limit:=${pi}
+     elbow_joint_lower_limit:=${-pi}    elbow_joint_upper_limit:=${pi}
+     wrist_1_lower_limit:=${-pi}    wrist_1_upper_limit:=${pi}
+     wrist_2_lower_limit:=${-pi}    wrist_2_upper_limit:=${pi}
+     wrist_3_lower_limit:=${-pi}    wrist_3_upper_limit:=${pi}">
     <!-- Inertia parameters -->
     <xacro:property name="base_mass" value="4.0" />  <!-- This mass might be incorrect -->
@@ -11,5 +27,5 @@
     <xacro:property name="wrist_2_mass" value="1.2190" />
     <xacro:property name="wrist_3_mass" value="0.1879" />
-     <xacro:property name="shoulder_cog" value="0.0 0.00193 -0.02561" />
+    <xacro:property name="shoulder_cog" value="0.0 0.00193 -0.02561" />
     <xacro:property name="upper_arm_cog" value="0.0 -0.024201 0.2125" />
     <xacro:property name="forearm_cog" value="0.0 0.0265 0.11993" />
@@ -17,5 +33,5 @@
     <xacro:property name="wrist_2_cog" value="0.0 0.0018 0.11099" />
     <xacro:property name="wrist_3_cog" value="0.0 0.001159 0.0" />
-     <!-- Kinematic model -->
+    <!-- Kinematic model -->
     <!-- Properties from urcontrol.conf -->
     <!--
@@ -35,8 +51,8 @@
     <xacro:property name="d5" value="0.09465" />
     <xacro:property name="d6" value="0.0823" />
-     <!-- Arbitrary offsets for shoulder/elbow joints -->
+    <!-- Arbitrary offsets for shoulder/elbow joints -->
     <xacro:property name="shoulder_offset" value="0.13585" />  <!-- measured from model -->
     <xacro:property name="elbow_offset" value="-0.1197" /> <!-- measured from model -->
-     <!-- link lengths used in model -->
+    <!-- link lengths used in model -->
     <xacro:property name="shoulder_height" value="${d1}" />
     <xacro:property name="upper_arm_length" value="${-a2}" />
@@ -53,33 +69,10 @@
     <!--property name="wrist_2_length" value="0.09465" /-->   <!-- In CAD this distance is 0.930, but in the spec it is 0.09465 -->
     <!--property name="wrist_3_length" value="0.0823" /-->
-     <xacro:property name="shoulder_radius" value="0.060" />   <!-- manually measured -->
+    <xacro:property name="shoulder_radius" value="0.060" />   <!-- manually measured -->
     <xacro:property name="upper_arm_radius" value="0.054" />  <!-- manually measured -->
     <xacro:property name="elbow_radius" value="0.060" />      <!-- manually measured -->
     <xacro:property name="forearm_radius" value="0.040" />    <!-- manually measured -->
     <xacro:property name="wrist_radius" value="0.045" />      <!-- manually measured -->
-  <xacro:macro name="cylinder_inertial" params="radius length mass *origin">
-    <inertial>
-      <mass value="${mass}" />
-      <xacro:insert_block name="origin" />
-      <inertia ixx="${0.0833333 * mass * (3 * radius * radius + length * length)}" ixy="0.0" ixz="0.0"
-        iyy="${0.0833333 * mass * (3 * radius * radius + length * length)}" iyz="0.0"
-        izz="${0.5 * mass * radius * radius}" />
-    </inertial>
-  </xacro:macro>
-  <xacro:macro name="ur5_robot" params="prefix joint_limited
-     shoulder_pan_lower_limit:=${-pi}    shoulder_pan_upper_limit:=${pi}
-     shoulder_lift_lower_limit:=${-pi}    shoulder_lift_upper_limit:=${pi}
-     elbow_joint_lower_limit:=${-pi}    elbow_joint_upper_limit:=${pi}
-     wrist_1_lower_limit:=${-pi}    wrist_1_upper_limit:=${pi}
-     wrist_2_lower_limit:=${-pi}    wrist_2_upper_limit:=${pi}
-     wrist_3_lower_limit:=${-pi}    wrist_3_upper_limit:=${pi}">
- <!--       new add       -->
-<!--   <origin xyz="0.28 0.0 0" rpy="0.0 0.0 -1.5708" />    -->
-  <joint name="ur_base_link_joint" type="fixed">
-    <origin xyz="0.28 0.0 0" rpy="0.0 0.0 ${-pi/4}" />
-    <parent link="mid_mount"/>
-    <child link="ur_base_link" />
-  </joint>
-    <link name="ur_base_link" >
+    <link name="${prefix}base_link" >
       <visual>
         <geometry>
@@ -100,5 +93,5 @@
     </link>
     <joint name="${prefix}shoulder_pan_joint" type="revolute">
-      <parent link="ur_base_link" />
+      <parent link="${prefix}base_link" />
       <child link = "${prefix}shoulder_link" />
       <origin xyz="0.0 0.0 ${shoulder_height}" rpy="0.0 0.0 0.0" />
@@ -136,5 +129,5 @@
       <axis xyz="0 1 0" />
       <xacro:unless value="${joint_limited}">
-        <limit lower="${pi/4}" upper="${3*pi / 4}" effort="150.0" velocity="3.15"/>
+        <limit lower="${-2.0 * pi}" upper="${2.0 * pi}" effort="150.0" velocity="3.15"/>
       </xacro:unless>
       <xacro:if value="${joint_limited}">
@@ -167,5 +160,5 @@
       <axis xyz="0 1 0" />
       <xacro:unless value="${joint_limited}">
-        <limit lower="${-3*pi / 4}" upper="${3*pi / 4}" effort="150.0" velocity="3.15"/>
+        <limit lower="${-pi}" upper="${pi}" effort="150.0" velocity="3.15"/>
       </xacro:unless>
       <xacro:if value="${joint_limited}">
@@ -198,5 +191,5 @@
       <axis xyz="0 1 0" />
       <xacro:unless value="${joint_limited}">
-        <limit lower="${-5.0 * pi / 4}" upper="${pi / 4}" effort="28.0" velocity="3.2"/>
+        <limit lower="${-2.0 * pi}" upper="${2.0 * pi}" effort="28.0" velocity="3.2"/>
       </xacro:unless>
       <xacro:if value="${joint_limited}">
@@ -229,5 +222,5 @@
       <axis xyz="0 0 1" />
       <xacro:unless value="${joint_limited}">
-        <limit lower="${10 * pi / 9.0}" upper="${2.0 * pi}" effort="28.0" velocity="3.2"/>
+        <limit lower="${-2.0 * pi}" upper="${2.0 * pi}" effort="28.0" velocity="3.2"/>
       </xacro:unless>
       <xacro:if value="${joint_limited}">
@@ -308,5 +301,5 @@
       -->
       <origin xyz="0 0 0" rpy="0 0 ${-pi}"/>
-      <parent link="ur_base_link"/>
+      <parent link="${prefix}base_link"/>
       <child link="${prefix}base"/>
     </joint>

File: ur_description/urdf/ur5_joint_limited_robot.urdf.xacro (robot description, xacro)
@@ -1,4 +1,4 @@
 <?xml version="1.0"?>
-<robot xmlns:xacro="http://www.ros.org/wiki/xacro"
+<robot xmlns:xacro="http://wiki.ros.org/xacro"
        name="ur5" >
   <!-- common stuff -->
@@ -15,11 +15,9 @@
     wrist_3_lower_limit="${-pi}" wrist_3_upper_limit="${pi}"
   />
-<!--
-  <link name="mid_mount_1" />
-  <joint name="mid_mount_joint_1" type="fixed">
-    <parent link="mid_mount" />
-    <child link = "mid_mount_1" />
+  <link name="world" />
+  <joint name="world_joint" type="fixed">
+    <parent link="world" />
+    <child link = "base_link" />
     <origin xyz="0.0 0.0 0.0" rpy="0.0 0.0 0.0" />
   </joint>
--->
 </robot>

File: ur_description/urdf/ur5_robot.urdf.xacro (robot description, xacro)
@@ -1,4 +1,4 @@
 <?xml version="1.0"?>
-<robot xmlns:xacro="http://www.ros.org/wiki/xacro"
+<robot xmlns:xacro="http://wiki.ros.org/xacro"
        name="ur5" >
   <!-- common stuff -->
